File: hw/RevA/RevA.sch (KiCad schematic (older format))
At the start: 116 parts, among them J1 USB_C_Receptacle_USB2.0, J3 DNP Conn_01x02, J4 DNP Conn_02x03_Odd_Even, SW1 SW_Push, U1 SY8120B1ABC, U2 XC6206P25, U3 SY8120B1ABC, U4 SPI Flash W25Q128JVSIQ, U8 LFE5U-12F-6BG256C, U9 16MHz 20ppm

Commit message: progress
Parts:
- gave numbers to parts that had none: 24

Commit message: progress
Parts:
- removed H1, H2, H3, H4: DNP, MountingHole:MountingHole_3.5mm, symbol Mechanical:MountingHole
- removed J4: DNP Conn_02x03_Odd_Even, Connector_PinHeader_2.54mm:PinHeader_2x03_P2.54mm_Vertical_SMD, symbol Connector_Generic:Conn_02x03_Odd_Even
- removed J5: Conn_UART, symbol Connector_Generic:Conn_01x03
- removed LOGO2: Logo_Open_Hardware_Small, ecp5board:logo, symbol Graphic:Logo_Open_Hardware_Small
- added DBG1: Conn_02x06_Top_Bottom, ecp5board:PMOD_Socket_2x06_P2.54mm_Horizontal, symbol Connector_Generic:Conn_02x06_Top_Bottom
- J2: footprint (none) -> Connector_Card:microSD_HC_Molex_104031-0811
- JP1: footprint ecp5board:JP_3_0402_1005Metric -> Connector_PinHeader_2.54mm:PinHeader_1x03_P2.54mm_Horizontal
- U6: footprint Package_SO:TSOP-II-54_10.16x22.22mm_P0.8mm -> Package_SO:TSOP-II-54_22.2x10.16mm_P0.8mm
- renumbered U5 to CON1
Connections:
- net labels added: DEBUG_1, DEBUG_2
Changed lines of the file:
@@
 $EndComp
 $Comp
-L Mechanical:MountingHole H1
-U 1 1 5DAC6FCA
-P 17800 15550
-F 0 "H1" H 17900 15596 50  0000 L CNN
-F 1 "DNP" H 17900 15505 50  0000 L CNN
-F 2 "MountingHole:MountingHole_3.5mm" H 17800 15550 50  0001 C CNN
-F 3 " " H 17800 15550 50  0001 C CNN
-	1    17800 15550
-	1    0    0    -1
-$EndComp
-$Comp
-L Mechanical:MountingHole H2
-U 1 1 5DAC7771
-P 17800 15750
-F 0 "H2" H 17900 15796 50  0000 L CNN
-F 1 "DNP" H 17900 15705 50  0000 L CNN
-F 2 "MountingHole:MountingHole_3.5mm" H 17800 15750 50  0001 C CNN
-F 3 " " H 17800 15750 50  0001 C CNN
-	1    17800 15750
-	1    0    0    -1
-$EndComp
-$Comp
-L Mechanical:MountingHole H4
-U 1 1 5DAC7F79
-P 18250 15750
-F 0 "H4" H 18350 15796 50  0000 L CNN
-F 1 "DNP" H 18350 15705 50  0000 L CNN
-F 2 "MountingHole:MountingHole_3.5mm" H 18250 15750 50  0001 C CNN
-F 3 " " H 18250 15750 50  0001 C CNN
-	1    18250 15750
-	1    0    0    -1
-$EndComp
-$Comp
-L Mechanical:MountingHole H3
-U 1 1 5DAC8373
-P 18250 15550
-F 0 "H3" H 18350 15596 50  0000 L CNN
-F 1 "DNP" H 18350 15505 50  0000 L CNN
-F 2 "MountingHole:MountingHole_3.5mm" H 18250 15550 50  0001 C CNN
-F 3 " " H 18250 15550 50  0001 C CNN
-	1    18250 15550
-	1    0    0    -1
-$EndComp
-$Comp
 L Lattice_ECP5_LFE5U-cabga256:LFE5U-12F-6BG256C U8
 U 1 1 5DB1D5C1
@@
 Wire Wire Line
 	1200 9200 1200 9250
-$Comp
-L Connector_Generic:Conn_02x03_Odd_Even J4
-U 1 1 5DEFDC14
-P 14150 1050
-F 0 "J4" H 14200 1367 50  0000 C CNN
-F 1 "DNP Conn_02x03_Odd_Even" H 14200 1276 50  0000 C CNN
-F 2 "Connector_PinHeader_2.54mm:PinHeader_2x03_P2.54mm_Vertical_SMD" H 14150 1050 50  0001 C CNN
-F 3 " " H 14150 1050 50  0001 C CNN
-	1    14150 1050
-	1    0    0    -1
-$EndComp
-$Comp
-L power:GND #PWR079
-U 1 1 5DEFFFD3
-P 13300 1350
-F 0 "#PWR079" H 13300 1100 50  0001 C CNN
-F 1 "GND" H 13305 1177 50  0000 C CNN
-F 2 "" H 13300 1350 50  0001 C CNN
-F 3 "" H 13300 1350 50  0001 C CNN
-	1    13300 1350
-	1    0    0    -1
-$EndComp
-Text Label 13750 1050 2    50   ~ 0
+Text Label 13800 1150 2    50   ~ 0
 JTAG_TDI
 Wire Wire Line
-	13750 1050 13950 1050
-Text Label 13750 1150 2    50   ~ 0
+	13800 1150 14000 1150
+Text Label 13800 850  2    50   ~ 0
 JTAG_TMS
 Wire Wire Line
-	13750 1150 13950 1150
-Text Label 14550 1050 0    50   ~ 0
+	13800 850  14000 850
+Text Label 13800 950  2    50   ~ 0
 JTAG_TCK
-Text Label 14550 1150 0    50   ~ 0
+Text Label 13800 1050 2    50   ~ 0
 JTAG_TDO
 Wire Wire Line
-	14550 1150 14450 1150
-Wire Wire Line
-	13300 950  13950 950
-Wire Wire Line
-	13300 950  13300 1350
-$Comp
-L power:+3V3 #PWR0105
-U 1 1 5DF7DEEE
-P 14650 850
-F 0 "#PWR0105" H 14650 700 50  0001 C CNN
-F 1 "+3V3" H 14665 1023 50  0000 C CNN
-F 2 "" H 14650 850 50  0001 C CNN
-F 3 "" H 14650 850 50  0001 C CNN
-	1    14650 850
-	1    0    0    -1
-$EndComp
-Wire Wire Line
-	14650 850  14650 950
-Wire Wire Line
-	14650 950  14450 950
+	13800 1050 14000 1050
 $Comp
 L Lattice_ECP5_LFE5U-cabga256:LFE5U-12F-6BG256C U8
@@
 	20050 11100 20050 11050
 Wire Wire Line
-	14450 1050 14550 1050
+	14000 950  13800 950
 Text Label 21450 7450 2    50   ~ 0
 LED0
@@
 $EndComp
 $Comp
-L Graphic:Logo_Open_Hardware_Small LOGO2
-U 1 1 5DE75DAA
-P 16750 15650
-F 0 "LOGO2" H 16750 15925 50  0001 C CNN
-F 1 "Logo_Open_Hardware_Small" H 16750 15425 50  0001 C CNN
-F 2 "ecp5board:logo" H 16750 15650 50  0001 C CNN
-F 3 "~" H 16750 15650 50  0001 C CNN
-	1    16750 15650
-	1    0    0    -1
-$EndComp
-$Comp
 L Graphic:Logo_Open_Hardware_Small LOGO3
 U 1 1 5DF8D651
@@
 Text Label 16250 12350 2    50   ~ 0
 FPGA_CCLK
-$Comp
-L Connector_Generic:Conn_01x03 J5
-U 1 1 61EFD140
-P 14150 1850
-F 0 "J5" H 14230 1892 50  0000 L CNN
-F 1 "Conn_UART" H 14230 1801 50  0000 L CNN
-F 2 "" H 14150 1850 50  0001 C CNN
-F 3 "~" H 14150 1850 50  0001 C CNN
-	1    14150 1850
-	1    0    0    -1
-$EndComp
-Text Label 13750 1750 2    50   ~ 0
+Text Label 14700 950  0    50   ~ 0
 UART_TX
-Text Label 13750 1850 2    50   ~ 0
+Text Label 14700 850  0    50   ~ 0
 UART_RX
-$Comp
-L power:GND #PWR0101
-U 1 1 61F018F9
-P 13750 2050
-F 0 "#PWR0101" H 13750 1800 50  0001 C CNN
-F 1 "GND" H 13755 1877 50  0000 C CNN
-F 2 "" H 13750 2050 50  0001 C CNN
-F 3 "" H 13750 2050 50  0001 C CNN
-	1    13750 2050
-	1    0    0    -1
-$EndComp
-Wire Wire Line
-	13750 1750 13950 1750
 Wire Wire Line
-	13750 1850 13950 1850
+	14700 950  14500 950
 Wire Wire Line
-	13750 1950 13950 1950
-Wire Wire Line
-	13750 2050 13750 1950
+	14700 850  14500 850
 Wire Wire Line
 	700  1450 700  5350
@@
 F 0 "JP1" H 3300 7324 50  0000 C CNN
 F 1 "4K7" H 3300 7233 50  0000 C CNN
-F 2 "ecp5board:JP_3_0402_1005Metric" H 3300 7100 50  0001 C CNN
+F 2 "Connector_PinHeader_2.54mm:PinHeader_1x03_P2.54mm_Horizontal" H 3300 7100 50  0001 C CNN
 F 3 " " H 3300 7100 50  0001 C CNN
 F 4 "C105871" H 3300 7100 50  0001 C CNN "LCSC"
@@
 F 0 "J2" H 13950 11017 50  0000 C CNN
 F 1 "Micro_SD_Card" H 13950 10926 50  0000 C CNN
-F 2 "" H 15150 10600 50  0001 C CNN
+F 2 "Connector_Card:microSD_HC_Molex_104031-0811" H 15150 10600 50  0001 C CNN
 F 3 "http://katalog.we-online.de/em/datasheet/693072010801.pdf" H 14000 10300 50  0001 C CNN
 	1    14000 10300
@@
 F 0 "U6" H 8800 9450 50  0000 C CNN
 F 1 "IS42S16320F-7TL" H 9100 9350 50  0000 C CNN
-F 2 "Package_SO:TSOP-II-54_10.16x22.22mm_P0.8mm" H 8300 8100 50  0001 C CNN
+F 2 "Package_SO:TSOP-II-54_22.2x10.16mm_P0.8mm" H 8300 8100 50  0001 C CNN
 F 3 "http://www.issi.com/WW/pdf/42-45S16400J.pdf" H 7700 9350 50  0001 C CNN
 	1    8300 8100
@@
 N64_VCC
 $Comp
-L N64:N64-Cartridge U5
+L N64:N64-Cartridge CON1
 U 1 1 63378C0C
 P 7050 13750
-F 0 "U5" H 7050 15250 60  0000 C CNN
+F 0 "CON1" H 7050 15250 60  0000 C CNN
 F 1 "N64-Cartridge" H 7050 15150 60  0000 C CNN
 F 2 "ecp5board:N64-Connector" H 7000 12700 60  0000 C CNN
@@
 Wire Wire Line
 	3000 7700 3300 7700
+$Comp
+L power:+3V3 #PWR0101
+U 1 1 61EDAE19
+P 13800 1350
+F 0 "#PWR0101" H 13800 1200 50  0001 C CNN
+F 1 "+3V3" V 13815 1478 50  0000 L CNN
+F 2 "" H 13800 1350 50  0001 C CNN
+F 3 "" H 13800 1350 50  0001 C CNN
+	1    13800 1350
+	0    -1   -1   0
+$EndComp
+Wire Wire Line
+	13800 1350 14000 1350
+$Comp
+L Connector_Generic:Conn_02x06_Top_Bottom DBG1
+U 1 1 6219762F
+P 14200 1050
+F 0 "DBG1" H 14250 1467 50  0000 C CNN
+F 1 "Conn_02x06_Top_Bottom" H 14250 1376 50  0000 C CNN
+F 2 "ecp5board:PMOD_Socket_2x06_P2.54mm_Horizontal" H 14200 1050 50  0001 C CNN
+F 3 " " H 14200 1050 50  0001 C CNN
+F 4 "C239357" H 14200 1050 50  0001 C CNN "LCSC"
+F 5 "0.1299" H 14200 1050 50  0001 C CNN "LCSC EUR"
+F 6 "https://lcsc.com/product-detail/Pin-Header-Female-Header_Changjiang-Connectors-A2541HWR-2x6P_C239357.html" H 14200 1050 50  0001 C CNN "LCSC URL"
+	1    14200 1050
+	1    0    0    -1
+$EndComp
+$Comp
+L power:+3V3 #PWR0105
+U 1 1 6234C908
+P 14700 1350
+F 0 "#PWR0105" H 14700 1200 50  0001 C CNN
+F 1 "+3V3" V 14715 1478 50  0000 L CNN
+F 2 "" H 14700 1350 50  0001 C CNN
+F 3 "" H 14700 1350 50  0001 C CNN
+	1    14700 1350
+	0    1    1    0
+$EndComp
+Wire Wire Line
+	14700 1350 14500 1350
+$Comp
+L power:GND #PWR0146
+U 1 1 623E040E
+P 14700 1250
+F 0 "#PWR0146" H 14700 1000 50  0001 C CNN
+F 1 "GND" V 14705 1122 50  0000 R CNN
+F 2 "" H 14700 1250 50  0001 C CNN
+F 3 "" H 14700 1250 50  0001 C CNN
+	1    14700 1250
+	0    -1   -1   0
+$EndComp
+Wire Wire Line
+	14500 1250 14700 1250
+Wire Wire Line
+	14500 1150 14700 1150
+Wire Wire Line
+	14500 1050 14700 1050
+$Comp
+L power:GND #PWR0149
+U 1 1 6262AD24
+P 13800 1250
+F 0 "#PWR0149" H 13800 1000 50  0001 C CNN
+F 1 "GND" V 13805 1122 50  0000 R CNN
+F 2 "" H 13800 1250 50  0001 C CNN
+F 3 "" H 13800 1250 50  0001 C CNN
+	1    13800 1250
+	0    1    1    0
+$EndComp
+Wire Wire Line
+	14000 1250 13800 1250
+Text Label 14700 1050 0    50   ~ 0
+DEBUG_1
+Text Label 14700 1150 0    50   ~ 0
+DEBUG_2
 $EndSCHEMATC

Commit message: progress
Parts:
- removed C4: 4u7, Capacitor_SMD:C_0402_1005Metric, symbol Device:C_Small
- removed RN12: 22R_x4, Resistor_SMD:R_Array_Convex_4x0603, symbol Device:R_Pack04
- added D1: 1N914, Diode_SMD:D_SOD-323_HandSoldering, symbol Diode:1N914
- added R38: 1K1, Resistor_SMD:R_0402_1005Metric, symbol Device:R
Connections:
- net labels added: USB_PULL_DP
- wire segments 680 -> 678
- no-connect marks 127 -> 125
Other:
- note added: "Drive USB_PULL_DP high to enable\nUSB 1.1 FullSpeed device mode"
- note removed: "TODO: Add pull ups"
- moved on the sheet: FB1, JP1, R17, R8
Changed lines of the file:
@@
 Connection ~ 2250 8200
 Connection ~ 2250 8400
-Text Label 3350 8400 0    50   ~ 0
+Text Label 3000 8400 0    50   ~ 0
 USB_DP
-Text Label 3350 8200 0    50   ~ 0
+Text Label 3000 8200 0    50   ~ 0
 USB_DM
 $Comp
 L Device:Ferrite_Bead FB1
 U 1 1 5DD4A9CC
-P 2600 7700
-F 0 "FB1" V 2450 7500 50  0000 L CNN
-F 1 "Ferrite_Bead" V 2500 7150 50  0000 L CNN
-F 2 "Inductor_SMD:L_0805_2012Metric" V 2530 7700 50  0001 C CNN
-F 3 " " H 2600 7700 50  0001 C CNN
-F 4 "C88993" H 2600 7700 50  0001 C CNN "LCSC"
-F 5 "https://lcsc.com/product-detail/Ferrite-Beads-And-Chips_muRata_BLM21PG220SN1D_22R-25_C88993.html" H 2600 7700 50  0001 C CNN "LCSC URL"
-F 6 "0.0183" H 2600 7700 50  0001 C CNN "LCSC EUR"
-	1    2600 7700
+P 1500 7150
+F 0 "FB1" V 1450 7250 50  0000 L CNN
+F 1 "Ferrite_Bead" V 1400 6600 50  0000 L CNN
+F 2 "Inductor_SMD:L_0805_2012Metric" V 1430 7150 50  0001 C CNN
+F 3 " " H 1500 7150 50  0001 C CNN
+F 4 "C88993" H 1500 7150 50  0001 C CNN "LCSC"
+F 5 "https://lcsc.com/product-detail/Ferrite-Beads-And-Chips_muRata_BLM21PG220SN1D_22R-25_C88993.html" H 1500 7150 50  0001 C CNN "LCSC URL"
+F 6 "0.0183" H 1500 7150 50  0001 C CNN "LCSC EUR"
+	1    1500 7150
 	0    1    1    0
 $EndComp
@@
 L power:VBUS #PWR01
 U 1 1 5DC5476C
-P 3000 7600
-F 0 "#PWR01" H 3000 7450 50  0001 C CNN
-F 1 "VBUS" H 3015 7773 50  0000 C CNN
-F 2 "" H 3000 7600 50  0001 C CNN
-F 3 "" H 3000 7600 50  0001 C CNN
-	1    3000 7600
+P 2450 7600
+F 0 "#PWR01" H 2450 7450 50  0001 C CNN
+F 1 "VBUS" H 2465 7773 50  0000 C CNN
+F 2 "" H 2450 7600 50  0001 C CNN
+F 3 "" H 2450 7600 50  0001 C CNN
+	1    2450 7600
 	1    0    0    -1
 $EndComp
@@
 Wire Wire Line
 	1400 6250 1400 6400
-Connection ~ 2300 4450
-Wire Wire Line
-	2300 4450 2300 4500
 $Comp
 L Device:C_Small C6
@@
 	13800 4250 13800 4300
 Wire Wire Line
-	700  7100 700  5350
+	700  7150 700  5350
 Connection ~ 700  5350
 Text Label 16800 4600 2    50   ~ 0
@@
 	1050 2500 1400 2500
 Connection ~ 1400 2500
-Wire Wire Line
-	1050 4250 1050 4450
 $Comp
 L Device:C_Small C1
@@
 	1000 6400 1400 6400
 Connection ~ 1400 6400
-Wire Wire Line
-	1050 3400 1050 4050
 Text Label 16850 11750 2    50   ~ 0
 FPGA_SPI_D0
@@
 $EndComp
 Wire Wire Line
-	2300 3700 2300 4450
-Wire Wire Line
 	2300 4500 4500 4500
 Wire Wire Line
 	2700 3400 4500 3400
 Wire Wire Line
-	1050 4450 2300 4450
-Wire Wire Line
 	1050 3400 1900 3400
-$Comp
-L Device:C_Small C4
-U 1 1 5DFFA7BA
-P 1050 4150
-F 0 "C4" H 958 4104 50  0000 R CNN
-F 1 "4u7" H 958 4195 50  0000 R CNN
-F 2 "Capacitor_SMD:C_0402_1005Metric" H 1050 4150 50  0001 C CNN
-F 3 " " H 1050 4150 50  0001 C CNN
-	1    1050 4150
-	-1   0    0    1
-$EndComp
 Text Notes 4900 3450 0    50   ~ 0
 2V5: 200mA max
@@
 RevA 0.1:\n
 $Sheet
-S 4000 8650 900  550
+S 2350 10400 900  550
 U 61266D88
 F0 "Overview" 50
@@
 	1    0    0    -1
 $EndComp
-Connection ~ 1050 3400
 Text Label 700  1300 0    50   ~ 0
 V_SUPPLY
@@
 L Jumper:Jumper_3_Open JP1
 U 1 1 6220D837
-P 3300 7100
-F 0 "JP1" H 3300 7324 50  0000 C CNN
-F 1 "4K7" H 3300 7233 50  0000 C CNN
-F 2 "Connector_PinHeader_2.54mm:PinHeader_1x03_P2.54mm_Horizontal" H 3300 7100 50  0001 C CNN
-F 3 " " H 3300 7100 50  0001 C CNN
-F 4 "C105871" H 3300 7100 50  0001 C CNN "LCSC"
-F 5 "0.0005" H 3300 7100 50  0001 C CNN "LCSC EUR"
-F 6 "https://lcsc.com/product-detail/Chip-Resistor-Surface-Mount_4-7KR-4701-1_C105871.html" H 3300 7100 50  0001 C CNN "LCSC URL"
-	1    3300 7100
-	0    1    1    0
+P 2800 7150
+F 0 "JP1" H 2800 7374 50  0000 C CNN
+F 1 "4K7" H 2800 7283 50  0000 C CNN
+F 2 "Connector_PinHeader_2.54mm:PinHeader_1x03_P2.54mm_Horizontal" H 2800 7150 50  0001 C CNN
+F 3 " " H 2800 7150 50  0001 C CNN
+F 4 "C105871" H 2800 7150 50  0001 C CNN "LCSC"
+F 5 "0.0005" H 2800 7150 50  0001 C CNN "LCSC EUR"
+F 6 "https://lcsc.com/product-detail/Chip-Resistor-Surface-Mount_4-7KR-4701-1_C105871.html" H 2800 7150 50  0001 C CNN "LCSC URL"
+	1    2800 7150
+	0    1    -1   0
 $EndComp
 $Comp
@@
 	8050 13750 8450 13750
 Wire Wire Line
-	8050 13850 8450 13850
-Wire Wire Line
 	8050 13950 8450 13950
 Wire Wire Line
@@
 	5600 13650 6000 13650
 Wire Wire Line
-	5600 13750 6000 13750
-Wire Wire Line
 	5600 13850 6000 13850
 Wire Wire Line
@@
 N64_ALEH
 NoConn ~ 8450 13750
-NoConn ~ 8450 13850
 Text Label 8450 14150 0    50   ~ 0
 N64_VCC
@@
 N64_VCC
 NoConn ~ 5600 13850
-NoConn ~ 5600 13750
 Text Label 5600 13450 2    50   ~ 0
 N64_READ
@@
 $EndComp
 $Comp
-L Device:R_Pack04 RN12
-U 1 1 666C0572
-P 10350 15750
-F 0 "RN12" V 10050 15750 50  0000 C CNN
-F 1 "22R_x4" V 10050 15800 50  0001 C CNN
-F 2 "Resistor_SMD:R_Array_Convex_4x0603" V 10625 15750 50  0001 C CNN
-F 3 " " H 10350 15750 50  0001 C CNN
-F 4 "C309446" V 10350 15750 50  0001 C CNN "LCSC"
-F 5 "0.0075" H 10350 15750 50  0001 C CNN "LCSC EUR"
-F 6 "https://lcsc.com/product-detail/Others_YAGEO-AF124-JR-0722RL_C309446.html" H 10350 15750 50  0001 C CNN "LCSC URL"
-	1    10350 15750
-	0    1    1    0
-$EndComp
-$Comp
 L Device:R_Pack04 RN10
 U 1 1 666C0560
@@
 Text Label 10050 15300 2    50   ~ 0
 N64_NMI
-Text Label 10050 15550 2    50   ~ 0
+Text Label 10050 13500 2    50   ~ 0
 N64_RAUDIO
 Wire Wire Line
@@
 Wire Wire Line
 	10050 15300 10150 15300
-Wire Wire Line
-	10050 15550 10150 15550
-Wire Wire Line
-	10050 15650 10150 15650
 $Comp
 L Device:R_Pack04 RN11
@@
 $EndComp
 NoConn ~ 16950 12050
-Text Notes 3800 8200 0    50   ~ 0
-TODO: Add pull ups
 $Comp
 L Device:R R17
 U 1 1 6A9F5C9D
-P 2850 8400
-F 0 "R17" V 2900 8250 50  0000 C CNN
-F 1 "22R" V 2850 8400 39  0000 C CNN
-F 2 "Resistor_SMD:R_0402_1005Metric" V 2780 8400 50  0001 C CNN
-F 3 " " H 2850 8400 50  0001 C CNN
-	1    2850 8400
+P 2550 8400
+F 0 "R17" V 2600 8150 50  0000 L CNN
+F 1 "22R" V 2550 8400 39  0000 C CNN
+F 2 "Resistor_SMD:R_0402_1005Metric" V 2480 8400 50  0001 C CNN
+F 3 " " H 2550 8400 50  0001 C CNN
+	1    2550 8400
 	0    -1   -1   0
 $EndComp
 Wire Wire Line
-	2250 8400 2700 8400
-Wire Wire Line
-	3000 8400 3350 8400
+	2250 8400 2400 8400
 $Comp
 L Device:R R8
 U 1 1 6AB1C912
-P 2850 8200
-F 0 "R8" V 2900 8050 50  0000 C CNN
-F 1 "22R" V 2850 8200 39  0000 C CNN
-F 2 "Resistor_SMD:R_0402_1005Metric" V 2780 8200 50  0001 C CNN
-F 3 " " H 2850 8200 50  0001 C CNN
-	1    2850 8200
+P 2550 8200
+F 0 "R8" V 2600 8000 50  0000 L CNN
+F 1 "22R" V 2550 8200 39  0000 C CNN
+F 2 "Resistor_SMD:R_0402_1005Metric" V 2480 8200 50  0001 C CNN
+F 3 " " H 2550 8200 50  0001 C CNN
+	1    2550 8200
 	0    -1   -1   0
 $EndComp
 Wire Wire Line
-	2250 8200 2700 8200
-Wire Wire Line
-	3000 8200 3350 8200
+	2250 8200 2400 8200
 Wire Wire Line
-	2100 7700 2450 7700
-Wire Wire Line
-	3300 6800 3300 6850
-Text Label 2450 7100 0    50   ~ 0
-V_SUPPLY
+	2700 8200 3000 8200
 Wire Wire Line
-	2750 7700 3000 7700
+	2800 6800 2800 6900
 Wire Wire Line
-	3300 7350 3300 7700
+	2800 7400 2800 7700
 $Comp
 L power:+12V #PWR0145
 U 1 1 6B7E33AE
-P 3300 6800
-F 0 "#PWR0145" H 3300 6650 50  0001 C CNN
-F 1 "+12V" H 3315 6973 50  0000 C CNN
-F 2 "" H 3300 6800 50  0001 C CNN
-F 3 "" H 3300 6800 50  0001 C CNN
-	1    3300 6800
+P 2800 6800
+F 0 "#PWR0145" H 2800 6650 50  0001 C CNN
+F 1 "+12V" H 2815 6973 50  0000 C CNN
+F 2 "" H 2800 6800 50  0001 C CNN
+F 3 "" H 2800 6800 50  0001 C CNN
+	1    2800 6800
 	1    0    0    -1
 $EndComp
 Wire Wire Line
-	700  7100 3150 7100
-Wire Wire Line
-	3000 7600 3000 7700
-Connection ~ 3000 7700
-Wire Wire Line
-	3000 7700 3300 7700
+	2450 7600 2450 7700
 $Comp
 L power:+3V3 #PWR0101
@@
 Text Label 14700 1150 0    50   ~ 0
 DEBUG_2
+Wire Wire Line
+	1350 7150 700  7150
+Wire Wire Line
+	2100 7700 2450 7700
+Wire Wire Line
+	2650 7150 1650 7150
+Wire Wire Line
+	2450 7700 2800 7700
+Connection ~ 2450 7700
+$Comp
+L Device:R R38
+U 1 1 61A3809E
+P 3550 8400
+F 0 "R38" V 3600 8150 50  0000 L CNN
+F 1 "1K1" V 3550 8400 39  0000 C CNN
+F 2 "Resistor_SMD:R_0402_1005Metric" V 3480 8400 50  0001 C CNN
+F 3 " " H 3550 8400 50  0001 C CNN
+	1    3550 8400
+	0    -1   -1   0
+$EndComp
+$Comp
+L Diode:1N914 D1
+U 1 1 6237C280
+P 4000 8400
+F 0 "D1" H 4000 8617 50  0000 C CNN
+F 1 "1N914" H 4000 8526 50  0000 C CNN
+F 2 "Diode_SMD:D_SOD-323_HandSoldering" H 4000 8225 50  0001 C CNN
+F 3 "http://www.vishay.com/docs/85622/1n914.pdf" H 4000 8400 50  0001 C CNN
+	1    4000 8400
+	1    0    0    -1
+$EndComp
+Wire Wire Line
+	3700 8400 3850 8400
+Text Label 4350 8400 0    50   ~ 0
+USB_PULL_DP
+Wire Wire Line
+	4350 8400 4150 8400
+Wire Wire Line
+	2700 8400 3400 8400
+Text Notes 3450 8150 0    50   ~ 0
+Drive USB_PULL_DP high to enable\nUSB 1.1 FullSpeed device mode
+$Comp
+L power:+12V #PWR0147
+U 1 1 62B7FE52
+P 9000 13750
+F 0 "#PWR0147" H 9000 13600 50  0001 C CNN
+F 1 "+12V" H 9015 13923 50  0000 C CNN
+F 2 "" H 9000 13750 50  0001 C CNN
+F 3 "" H 9000 13750 50  0001 C CNN
+	1    9000 13750
+	1    0    0    -1
+$EndComp
+Wire Wire Line
+	9000 13750 9000 13850
+Wire Wire Line
+	8050 13850 9000 13850
+$Comp
+L power:+12V #PWR0148
+U 1 1 62C157A8
+P 5000 13650
+F 0 "#PWR0148" H 5000 13500 50  0001 C CNN
+F 1 "+12V" H 5015 13823 50  0000 C CNN
+F 2 "" H 5000 13650 50  0001 C CNN
+F 3 "" H 5000 13650 50  0001 C CNN
+	1    5000 13650
+	1    0    0    -1
+$EndComp
+Wire Wire Line
+	5000 13750 5000 13650
+Wire Wire Line
+	5000 13750 6000 13750
+Wire Wire Line
+	2300 3700 2300 4500
 $EndSCHEMATC

Commit message: WIP
Connections:
- net labels added: N64_INT1
- no-connect marks 125 -> 124
Changed lines of the file:
@@
 F 6 "https://lcsc.com/product-detail/Chip-Resistor-Surface-Mount_4-7KR-4701-1_C105871.html" H 2800 7150 50  0001 C CNN "LCSC URL"
 	1    2800 7150
-	0    1    -1   0
+	0    1    1    0
 $EndComp
 $Comp
@@
 Text Label 8450 14250 0    50   ~ 0
 N64_CIC_DCLK
-NoConn ~ 8450 14350
 Text Label 8450 14450 0    50   ~ 0
 N64_NMI
@@
 F 0 "CON1" H 7050 15250 60  0000 C CNN
 F 1 "N64-Cartridge" H 7050 15150 60  0000 C CNN
-F 2 "ecp5board:N64-Connector" H 7000 12700 60  0000 C CNN
+F 2 "ecp5board:N64-Connector" H 7050 12400 60  0000 C CNN
 F 3 "" H 7000 12700 60  0000 C CNN
 	1    7050 13750
@@
 Wire Wire Line
 	2300 3700 2300 4500
+Text Label 8450 14350 0    50   ~ 0
+N64_INT1
 $EndSCHEMATC
